Commit message: Add existing project files prior to the push to GitHub.

File: description/robot.urdf.xacro (robot description, xacro)
@@ -2,3 +2,8 @@
 <robot xmlns:xacro="http://www.ros.org/wiki/xacro"  name="robot">
     <xacro:include filename="robot_core.xacro"/>
+    <!-- <xacro:include filename="gazebo_control.xacro"/> -->
+    <xacro:include filename="ros2_control.xacro"/>
+    <xacro:include filename = "lidar.xacro"/>
+    <!--xacro:include filename = "camera.xacro"/-->
+    <xacro:include filename = "depth_camera.xacro"/>
 </robot>

File: description/robot_core.xacro (robot description, xacro)
@@ -16,4 +16,12 @@
     <!-- Base Link -->
     <link name="base_link">
+    </link>
+    <!--Base Footprint Link-->
+    <joint name="base_footprint_joint" type="fixed">
+        <origin xyz="0.0 0.0 0.0" rpy="0.0 0.0 0.0"/>
+        <parent link="base_link"/>
+        <child link="base_footprint"/>
+    </joint>
+    <link name="base_footprint">
     </link>
     <!-- Chassis joint  -->
@@ -43,4 +51,7 @@
         </xacro:inertial_box>
     </link>
+    <gazebo reference="chassis">
+        <material>Gazebo/Red</material>
+    </gazebo>
     <!-- Left Wheel Link -->
     <joint name="left_wheel_joint" type="continuous">
@@ -68,4 +79,7 @@
         </xacro:inertial_cylinder>
     </link>
+    <gazebo reference="left_wheel">
+        <material>Gazebo/Blue</material>
+    </gazebo>
     <!-- Right Wheel Link -->
     <joint name="right_wheel_joint" type="continuous">
@@ -93,4 +107,7 @@
         </xacro:inertial_cylinder>
     </link>
+    <gazebo reference="right_wheel">
+        <material>Gazebo/Blue</material>
+    </gazebo>
     <!-- Caster wheel -->
     <joint name="caster_wheel_joint" type="fixed">
@@ -115,3 +132,8 @@
         </xacro:inertial_sphere>
     </link>
+    <gazebo reference="caster_wheel">
+        <material>Gazebo/Black</material>
+        <mu1 value="0.0001"/>
+        <mu2 value="0.0001"/>
+    </gazebo>
 </robot>
