Commit message: 19 Dec 2023

File: description/gazebo_control.xacro (robot description, xacro)
@@ -6,6 +6,6 @@
             <left_joint>left_wheel_joint</left_joint>
             <right_joint>right_wheel_joint</right_joint>
-            <wheel_separation>0.35</wheel_separation>
-            <wheel_diameter>0.1</wheel_diameter>
+            <wheel_separation>0.375</wheel_separation>
+            <wheel_diameter>0.065</wheel_diameter>
             <!-- Limits -->
             <max_wheel_torque>200</max_wheel_torque>

File: description/lidar.xacro (robot description, xacro)
@@ -4,10 +4,10 @@
         <parent link="chassis"/>
         <child link="laser_frame"/>
-        <origin xyz="0.1 0.0 0.175" rpy="0.0 0.0 0.0"/>
+        <origin xyz="0.3 0.0 0.145" rpy="0.0 0.0 0.0"/>
     </joint>
     <link name="laser_frame">
         <visual>
             <geometry>
-                <cylinder radius="0.05" length="0.04"/>
+                <cylinder radius="0.035" length="0.05"/>
             </geometry>
             <material name="black"/>
@@ -15,8 +15,8 @@
         <collision>
             <geometry>
-                <cylinder radius="0.05" length="0.04"/>
+                <cylinder radius="0.035" length="0.05"/>
             </geometry>
         </collision>
-        <xacro:inertial_cylinder mass="0.1" length="0.04" radius="0.05">
+        <xacro:inertial_cylinder mass="0.1" length="0.05" radius="0.035">
             <origin xyz="0 0 0" rpy="0 0 0"/>
         </xacro:inertial_cylinder>

File: description/robot_core.xacro (robot description, xacro)
@@ -34,7 +34,7 @@
     <link name= "chassis">
         <visual>
-            <origin xyz="0.15 0 0.075"/>
+            <origin xyz="0.165 0 0.075"/>
             <geometry>
-                <box size="0.3 0.3 0.15"/>
+                <box size="0.418 0.352 0.095"/>
                 <material name ="white"/>
             </geometry>
@@ -43,5 +43,5 @@
             <origin xyz="0.15 0 0.075"/>
             <geometry>
-                <box size="0.3 0.3 0.15"/>
+                <box size="0.418 0.352 0.95"/>
                 <material name ="white"/>
             </geometry>
@@ -56,5 +56,5 @@
     <!-- Left Wheel Link -->
     <joint name="left_wheel_joint" type="continuous">
-        <origin xyz="0 0.175 0" rpy="-${pi/2} 0.0 0.0"/>
+        <origin xyz="0 0.200 0" rpy="-${pi/2} 0.0 0.0"/>
         <parent link="base_link"/>
         <child link="left_wheel"/>
@@ -65,5 +65,33 @@
             <origin xyz="0.0 0.0 0.0" rpy="0.0 0.0 0.0"/>
             <geometry>
-                <cylinder radius="0.05" length="0.04"/>
+                <cylinder radius="0.0325" length="0.026"/>
+            </geometry>
+            <material name="blue"/>
+        </visual>
+        <collision>
+            <origin xyz="0.0 0.0 0.0" rpy="0.0 0.0 0.0"/>
+            <geometry>
+                <cylinder radius="0.0325" length="0.026"/>
+            </geometry>
+        </collision>
+        <xacro:inertial_cylinder mass="0.1" length="0.026" radius="0.0325">
+            <origin xyz="0 0 0" rpy="0 0 0"/>
+        </xacro:inertial_cylinder>
+    </link>
+    <gazebo reference="left_wheel">
+        <material>Gazebo/Blue</material>
+    </gazebo>
+    <!-- Right Wheel Link -->
+    <joint name="right_wheel_joint" type="continuous">
+        <origin xyz="0 -0.200 0" rpy="${pi/2} 0.0 0.0"/>
+        <parent link="base_link"/>
+        <child link="right_wheel"/>
+        <axis xyz="0.0 0.0 -1"/>
+    </joint>
+    <link name="right_wheel">
+        <visual name="">
+            <origin xyz="0.0 0.0 0.0" rpy="0.0 0.0 0.0"/>
+            <geometry>
+                <cylinder radius="0.0325" length="0.026"/>
             </geometry>
             <material name="blue"/>
@@ -75,33 +103,5 @@
             </geometry>
         </collision>
-        <xacro:inertial_cylinder mass="0.1" length="0.04" radius="0.05">
-            <origin xyz="0 0 0" rpy="0 0 0"/>
-        </xacro:inertial_cylinder>
-    </link>
-    <gazebo reference="left_wheel">
-        <material>Gazebo/Blue</material>
-    </gazebo>
-    <!-- Right Wheel Link -->
-    <joint name="right_wheel_joint" type="continuous">
-        <origin xyz="0 -0.175 0" rpy="${pi/2} 0.0 0.0"/>
-        <parent link="base_link"/>
-        <child link="right_wheel"/>
-        <axis xyz="0.0 0.0 -1"/>
-    </joint>
-    <link name="right_wheel">
-        <visual name="">
-            <origin xyz="0.0 0.0 0.0" rpy="0.0 0.0 0.0"/>
-            <geometry>
-                <cylinder radius="0.05" length="0.04"/>
-            </geometry>
-            <material name="blue"/>
-        </visual>
-        <collision>
-            <origin xyz="0.0 0.0 0.0" rpy="0.0 0.0 0.0"/>
-            <geometry>
-                <cylinder radius="0.05" length="0.04"/>
-            </geometry>
-        </collision>
-        <xacro:inertial_cylinder mass="0.1" length="0.04" radius="0.05">
+        <xacro:inertial_cylinder mass="0.1" length="0.026" radius="0.0325">
             <origin xyz="0 0 0" rpy="0 0 0"/>
         </xacro:inertial_cylinder>
@@ -112,5 +112,5 @@
     <!-- Caster wheel -->
     <joint name="caster_wheel_joint" type="fixed">
-        <origin xyz="0.24 0.0 0.0" />
+        <origin xyz="0.325 0.0 0.0" />
         <parent link="chassis"/>
         <child link="caster_wheel"/>
@@ -119,5 +119,5 @@
         <visual name="">
             <geometry>
-                    <sphere radius="0.05"/>
+                    <sphere radius="0.0325"/>
             </geometry>
             <material name="black"/>
@@ -125,8 +125,8 @@
         <collision>
             <geometry>
-                    <sphere radius="0.05"/>
+                    <sphere radius="0.0325"/>
             </geometry>
         </collision>
-        <xacro:inertial_sphere mass="0.1" radius="0.05">
+        <xacro:inertial_sphere mass="0.1" radius="0.0325">
             <origin xyz="0 0 0" rpy="0 0 0"/>
         </xacro:inertial_sphere>
